Commit message: init

File: src/robot_sim_demo/urdf/campus_patrol_robot.urdf (robot description, URDF)
Before this commit: robot campus_patrol_robot, 7 links, 6 joints
Links:
- removed link caster_link
- added link caster_back_link, mass 0.005
- added link imu_link
- link base_link: mass 5.0 -> 0.82573504; geometry collision cylinder length=0.065 radius=0.089; visual mesh filename=package://robot_sim_demo/models/turtlebot3_burger/meshes/bu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 scale=0.001 0.001 0.001
- link camera_link: mass None -> 0.02; geometry 
- link laser_link: mass None -> 0.114; geometry visual mesh filename=package://robot_sim_demo/models/turtlebot3_burger/meshes/ld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 scale=0.001 0.001 0.001
- link wheel_left_link: mass 0.25 -> 0.02849894; geometry visual mesh filename=package://robot_sim_demo/models/turtlebot3_burger/meshes/le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 scale=0.001 0.001 0.001
- link wheel_right_link: mass 0.25 -> 0.02849894; geometry visual mesh filename=package://robot_sim_demo/models/turtlebot3_burger/meshes/ri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 scale=0.001 0.001 0.001
Joints:
- removed joint caster_joint
- removed joint laser_joint
- added joint caster_back_joint: type fixed, parent base_link, child caster_back_link, origin xyz=-0.081 0 -0.004 rpy=0 0 0
- added joint imu_joint: type fixed, parent base_link, child imu_link, origin xyz=-0.032 0 0.068 rpy=0 0 0
- added joint scan_joint: type fixed, parent base_link, child laser_link, origin xyz=-0.032 0 0.162 rpy=0 0 0
- joint base_joint: origin xyz=0 0 0.145 rpy=0 0 0 -> xyz=0.0 0.0 0.010 rpy=0 0 0
- joint camera_joint: origin xyz=0.31 0 0.20 rpy=0 0 0 -> xyz=0.045 0 0.120 rpy=0 0 0
- joint wheel_left_joint: origin xyz=0 0.20 -0.08 rpy=-1.5708 0 0 -> xyz=0.0 0.08 0.023 rpy=-1.57 0 0
- joint wheel_right_joint: origin xyz=0 -0.20 -0.08 rpy=-1.5708 0 0 -> xyz=0.0 -0.080 0.023 rpy=-1.57 0 0
