Commit message: docs: deliver K3 chapter 1 and linked runtime evidence
Signed-off-by: DuoQilai <duoqilai@outlook.com>

File: src/robot_sim_demo/urdf/turtlebot3_burger.urdf (robot description, URDF)
Before this commit: robot turtlebot3_burger, 8 links, 7 joints
Links:
- added link camera_optical_frame
Joints:
- added joint camera_optical_joint: type fixed, parent camera_link, child camera_optical_frame, origin xyz=0.020 0 0 rpy=-1.5707963267948966 0 -1.5707963267948966

Commit message: refactor: separate K3 chapter 1 sources and course documents
Signed-off-by: DuoQilai <duoqilai@outlook.com>

File: src/robot_sim_demo/urdf/turtlebot3_burger.urdf (robot description, URDF)
Before this commit: robot turtlebot3_burger, 9 links, 8 joints
Links:
- removed link camera_optical_frame
Joints:
- removed joint camera_optical_joint
